File: OpenBCI_ESP32_INPUT/ADS1299.kicad_sch (KiCad schematic)
At the start: 30 parts, among them J2 Conn_02x08_Odd_Even, J3 Conn_02x03_Odd_Even, J4 Conn_02x02_Odd_Even, U7 ADS1299IPAG1

Commit message: Code and STL updates
Parts:
- C25, C27, C29, C31: value 1u -> 0.1u
- C26, C28, C30, C32: value 0.1u -> 1u
Connections:
- net VREF: no longer names the net of C22.1, C23.1, U7.24 (VREFP)
